File: KiCAD/button_bar.sch (KiCad schematic (older format))
At the start: 12 parts, among them K1 CONN_3, SW1 SW_PUSH, SW2 SW_PUSH, SW3 SW_PUSH, SW4 SW_PUSH, SW5 SW_PUSH

Commit message: button board schematic update
Parts:
- removed K1: CONN_3, symbol CONN_3
- added C1: 100n, C2, symbol C
- added P1: Buttons, SIL-4, symbol CONN_4
- added SW6: RESET, SW-PB, symbol SW_PUSH
- R1, R10: footprint (none) -> RC03
- R2, R3, R4, R5: renamed from R?; footprint (none) -> RC03
- SW1: value SW_PUSH -> SW_UP; footprint (none) -> SW-PB
- SW2: value SW_PUSH -> SW_DN; footprint (none) -> SW-PB
- SW3: value SW_PUSH -> SW_OK; footprint (none) -> SW-PB
- SW4: value SW_PUSH -> SW_LT; footprint (none) -> SW-PB
- SW5: value SW_PUSH -> SW_RT; footprint (none) -> SW-PB
Connections:
- net labels added: PWR, RST
- wire segments 25 -> 34
Other:
- moved on the sheet: R1, SW1, SW2, SW3, SW4, SW5
